File: RFSoC_Frontend_v0.1/RFSoC_Frontend_v0.1.kicad_pcb (KiCad board)
At the start: 4 copper layers, 242.3 x 70.5 mm, 130 parts, among them J1 Conn_Coaxial, J10 LPAM-40-01.0-X-08-X-K-TR, J13 Conn_Coaxial, J14 Conn_Coaxial, J15 Conn_Coaxial, J16 Conn_Coaxial, J17 Conn_Coaxial, J18 Conn_Coaxial, J19 Conn_Coaxial, J2 Conn_Coaxial, J20 Conn_Coaxial, J3 Conn_Coaxial, J4 Conn_Coaxial, J5 Conn_Coaxial, J6 Conn_Coaxial, J7 Conn_Coaxial, J8 Conn_Coaxial, J9 LPAM-40-01.0-X-08-X-K-TR, U1 TCM2-33WX+, U10 TCM2-33WX+, U11 TCM2-33WX+, U12 TCM2-33WX+, U13 TCM2-33WX+, U14 TCM2-33WX+, U15 TCM2-33WX+, U16 TCM2-33WX+, U2 TCM2-33WX+, U3 TCM2-33WX+, U4 TCM2-33WX+, U5 TCM2-33WX+, U6 TCM2-33WX+, U7 TCM2-33WX+, U8 TCM2-33WX+, U9 TCM2-33WX+

Commit message: resize board
Parts:
- removed C17, C18, C19, C20, C21, C22, C23, C24, C25, C26, C27, C28, C29, C30, C31, C32: .01u, Capacitor_SMD:C_0402_1005Metric
- removed J13, J14, J15, J16, J17, J18, J19, J20: Conn_Coaxial, Connector_Coaxial:SMA_Amphenol_132289_EdgeMount
- removed R33, R34, R35, R36, R45, R46, R47, R48, R49, R50, R51, R52, R61, R62, R63, R64: 590, Resistor_SMD:R_0402_1005Metric
- removed R37, R38, R39, R40, R41, R42, R43, R44, R53, R54, R55, R56, R57, R58, R59, R60: 17.4, Resistor_SMD:R_0402_1005Metric
- removed U10, U11, U12, U13, U14, U15, U16, U9: TCM2-33WX+, MINICIRCUITS:XFMR_TCM2-33WX+
- moved J3 70.1 mm to (163.0, 82.3)
- moved U3 70.1 mm to (161.4, 73.1)
- moved C5 70.1 mm to (162.1, 69.3)
- moved C6 70.1 mm to (161.1, 69.3)
- moved R10 70.1 mm to (161.1, 65.7)
- moved R15 70.1 mm to (161.6, 67.5)
- moved R9 70.1 mm to (162.1, 65.7)
- moved R3 70.1 mm to (161.6, 63.9)
- moved J1 43.5 mm to (205.7, 83.0)
- moved C1 43.5 mm to (204.6, 70.1)
- moved C2 43.5 mm to (203.6, 70.1)
- moved R1 43.5 mm to (204.1, 64.7)
- moved R13 43.5 mm to (204.1, 68.3)
- moved R5 43.5 mm to (204.6, 66.5)
- moved R6 43.5 mm to (203.6, 66.5)
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Routing:
- net DAC_B1_N: track 9.50 -> 2.54 mm
- net DAC_B1_P: track 9.62 -> 2.84 mm
- net ADC_B1_N: track 7.31 -> 2.28 mm
- net ADC_B1_P: track 7.12 -> 2.28 mm
- net DAC_B0_N: track 3.93 -> 2.59 mm
- net ADC_B0_P: track 4.09 -> 2.85 mm
- net ADC_B0_N: track 3.71 -> 2.47 mm
- net DAC_A1_P: track 3.50 -> 2.54 mm
- net DAC_A0_N: track 3.56 -> 2.79 mm
- net DAC_B0_P: track 3.52 -> 2.89 mm
- net DAC_A0_P: track 3.37 -> 2.79 mm
- net DAC_A1_N: track 3.12 -> 2.54 mm
Other:
- board size 242.3 x 70.5 mm -> 191.5 x 45.1 mm

Commit message: route differential lines
Routing:
- net DAC_B1_N: track 2.54 -> 30.4 mm
- net DAC_B1_P: track 2.84 -> 30.2 mm
- net ADC_B0_N: track 2.47 -> 28.6 mm
- net ADC_A0_N: track 3.19 -> 28.8 mm, vias 1 -> 2
- net DAC_A1_N: track 2.54 -> 27.8 mm
- net ADC_B0_P: track 2.85 -> 27.7 mm
- net ADC_A0_P: track 3.19 -> 27.9 mm, vias 1 -> 2
- net DAC_A1_P: track 2.54 -> 26.9 mm
- net ADC_A1_N: track 3.74 -> 16.3 mm, vias 1 -> 2
- net ADC_B1_N: track 2.28 -> 14.6 mm
- net DAC_B0_N: track 2.59 -> 14.7 mm
- net DAC_A0_N: track 2.79 -> 14.7 mm
- net ADC_A1_P: track 2.47 -> 14.2 mm, vias 1 -> 2
- net ADC_B1_P: track 2.28 -> 13.5 mm
- net DAC_B0_P: track 2.89 -> 14.0 mm
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- added copper zone on F.Cu, net GND
Other:
- outline, holes or cut-outs redrawn
- board text added: "Notes : Check Breakout Mounting Hole screw sizes"
