File: RFSoC_Frontend/FMC_0.kicad_sch (KiCad schematic)
At the start: 4 parts, among them J9 LPAM-40-01.0-X-08-X-K-TR

Commit message: Finished Updated ADC schematic
ADC schematic was modified to match the pin map between
the rfsoc and the xm500.
Connections:
- net ADC_A0_N: now also J9.G09; no longer J9.A09
- net ADC_A0_P: now also J9.F09; no longer J9.B09
- net ADC_A1_N: now also J9.C10; no longer J9.A10
- net ADC_B0_N: now also J9.G12; no longer J9.A12
- net ADC_B0_P: now also J9.F12; no longer J9.B12
- net ADC_B1_N: now also J9.C13; no longer J9.A13
- net ADC_C0_N: now also J9.G15; no longer J9.A15
- net ADC_C0_P: now also J9.F15; no longer J9.B15
- net ADC_C1_N: now also J9.C16; no longer J9.A16
- net ADC_D0_N: now also J9.G18; no longer J9.A18
- net ADC_D0_P: now also J9.F18; no longer J9.B18
- net ADC_D1_N: now also J9.C19; no longer J9.A19
- net GND: now also J9.A01, J9.A03, J9.A05, J9.B02, J9.B04, J9.B06, J9.B07, J9.B22, J9.B23, J9.B25, J9.B26, J9.B28, J9.B29, J9.B31, J9.B32, J9.B34, J9.B35, J9.B37, J9.B38, J9.B40, J9.C01, J9.C03, J9.C05, J9.C08, J9.C09, J9.C11, J9.C12, J9.C14, J9.C15, J9.C17, J9.C18, J9.C20, J9.C22, J9.C23, J9.C25, J9.C26, J9.C28, J9.C29, J9.C31, J9.C32, J9.C34, J9.C35, J9.C37, J9.C38, J9.C40, J9.D02, J9.D04, J9.D06, J9.D08, J9.D09, J9.D10, J9.D11, J9.D12, J9.D13, J9.D14, J9.D15, J9.D16, J9.D17, J9.D18, J9.D19, J9.D20, J9.D22, J9.D23, J9.D24, J9.D25, J9.D26, J9.D27, J9.D28, J9.D29, J9.D30, J9.D31, J9.D32, J9.D33, J9.D34, J9.D35, J9.D36, J9.D37, J9.D38, J9.D39, J9.D40, J9.E01, J9.E03, J9.E05, J9.E08, J9.E09, J9.E10, J9.E11, J9.E12, J9.E13, J9.E14, J9.E15, J9.E16, J9.E17, J9.E18, J9.E19, J9.E20, J9.E22, J9.E23, J9.E24, J9.E25, J9.E26, J9.E27, J9.E28, J9.E29, J9.E30, J9.E31, J9.E32, J9.E33, J9.E34, J9.E35, J9.E36, J9.E37, J9.E38, J9.E39, J9.E40, J9.F02, J9.F04, J9.F06, J9.F08, J9.F10, J9.F11, J9.F13, J9.F14, J9.F16, J9.F17, J9.F19, J9.F20, J9.F22, J9.F24, J9.F25, J9.F27, J9.F28, J9.F30, J9.F31, J9.F33, J9.F34, J9.F36, J9.F37, J9.F39, J9.F40, J9.G01, J9.G03, J9.G05, J9.G08, J9.G10, J9.G11, J9.G13, J9.G14, J9.G16, J9.G17, J9.G19, J9.G20, J9.G22, J9.G24, J9.G25, J9.G27, J9.G28, J9.G30, J9.G31, J9.G33, J9.G34, J9.G36, J9.G37, J9.G39, J9.G40, J9.H02, J9.H04, J9.H06, J9.H08, J9.H09, J9.H10, J9.H11, J9.H12, J9.H13, J9.H14, J9.H15, J9.H16, J9.H17, J9.H18, J9.H19, J9.H20, J9.H22, J9.H23, J9.H24, J9.H25, J9.H26, J9.H27, J9.H28, J9.H29, J9.H30, J9.H31, J9.H32, J9.H33, J9.H34, J9.H35, J9.H36, J9.H37, J9.H38, J9.H39, J9.H40; no longer J9.A08, J9.A08, J9.A08, J9.A09, J9.A09, J9.A10, J9.A10, J9.A11, J9.A11, J9.A11, J9.A12, J9.A12, J9.A13, J9.A13, J9.A14, J9.A14, J9.A14, J9.A15, J9.A15, J9.A16, J9.A16, J9.A17, J9.A17, J9.A17, J9.A18, J9.A18, J9.A19, J9.A19, J9.A20, J9.A20, J9.A20, J9.A21, J9.A22, J9.A23, J9.A24, J9.A25, J9.A26, J9.A27, J9.A28, J9.A29, J9.A30, J9.A31, J9.A32, J9.A33, J9.A34, J9.A35, J9.A36, J9.A37, J9.A38, J9.A39, J9.A40, J9.B08, J9.B08, J9.B08, J9.B09, J9.B09, J9.B10, J9.B10, J9.B10, J9.B11, J9.B11, J9.B11, J9.B12, J9.B12, J9.B13, J9.B13, J9.B13, J9.B14, J9.B14, J9.B14, J9.B15, J9.B15, J9.B16, J9.B16, J9.B16, J9.B17, J9.B17, J9.B17, J9.B18, J9.B18, J9.B19, J9.B19, J9.B19, J9.B20, J9.B20, J9.B20, J9.B21, J9.B22, J9.B22, J9.B23, J9.B23, J9.B24, J9.B24, J9.B25, J9.B25, J9.B26, J9.B26, J9.B27, J9.B27, J9.B28, J9.B28, J9.B29, J9.B29, J9.B30, J9.B30, J9.B31, J9.B31, J9.B32, J9.B32, J9.B33, J9.B33, J9.B34, J9.B34, J9.B35, J9.B35, J9.B36, J9.B36, J9.B37, J9.B37, J9.B38, J9.B38, J9.B39, J9.B39, J9.B40, J9.B40
- net ADCIO_00: now reaches J9.A02
- net ADCIO_01: now reaches J9.A04
- net VCC1V8_BUS: now reaches J9.A06
- net VCC1V8_BUS: now also J9.C06
- net UTIL_3V3: now reaches J9.A07
- net UTIL_3V3: now also J9.C07, J9.D07, J9.E07, J9.F07, J9.G07, J9.H07
- net VCM01_224: now reaches J9.A21
- net ADCIO_02: now reaches J9.B01
- net ADCIO_03: now reaches J9.B03
- net ADCIO_05: now reaches J9.B05
- net ADCIO_05: now also J9.C02
- net ADC_CLKIN_0_N: now reaches J9.B36
- net ADC_CLKIN_2_N: now reaches J9.B39
- new net ADCIO_06: J9.C04
- new net ADCIO_07: J9.D01
- new net ADCIO_08: J9.D03
- new net ADCIO_09: J9.D05
- new net ADCIO_10: J9.E02
- new net ADCIO_11: J9.E04
- new net ADCIO_12: J9.F01
- new net ADCIO_13: J9.F03
- new net ADCIO_14: J9.F05
- new net ADCIO_15: J9.G02
- new net ADCIO_16: J9.G04
- new net ADCIO_17: J9.H01
- new net ADCIO_18: J9.H03
- new net ADCIO_19: J9.H05
- new net ADC_CLKIN_0_P: J9.C36
- new net ADC_CLKIN_1_N: J9.F35
- new net ADC_CLKIN_1_P: J9.G35
- new net ADC_CLKIN_2_P: J9.C39
- new net ADC_CLKIN_3_N: J9.F38
- new net ADC_CLKIN_3_P: J9.G38
- new net RFMC_I2C_SCL: J9.G06
- new net RFMC_I2C_SDA: J9.E06
- new net VCM01_225: J9.C21
- new net VCM01_226: J9.E21
- new net VCM01_227: J9.G21
- new net VCM23_224: J9.B21
- new net VCM23_225: J9.D21
- new net VCM23_226: J9.F21
- new net VCM23_227: J9.H21
- no-connect marks 3 -> 63
Other:
- title: (none) -> ADC CONNECTOR
- moved on the sheet: J9A, J9B, J9C, J9D
