File: RFSoC_Frontend/FMC_1.kicad_sch (KiCad schematic)
At the start: 4 parts, among them J10 LPAM-40-01.0-X-08-X-K-TR

Commit message: updated all
Connections:
- net DAC_A0_N: now also J10.C19; no longer J10.A19
- net DAC_A1_N: now also J10.G20; no longer J10.A20
- net DAC_A1_P: now also J10.F20; no longer J10.B20
- net DAC_B0_N: now also J10.C16; no longer J10.A16
- net DAC_B1_N: now also J10.G17; no longer J10.A17
- net DAC_B1_P: now also J10.F17; no longer J10.B17
- net GND: now also J10.A36, J10.A38, J10.A40, J10.B02, J10.B03, J10.B05, J10.B06, J10.B08, J10.B09, J10.B11, J10.B12, J10.B29, J10.B30, J10.B32, J10.B33, J10.B35, J10.B37, J10.B39, J10.C02, J10.C03, J10.C05, J10.C06, J10.C08, J10.C09, J10.C11, J10.C12, J10.C14, J10.C15, J10.C17, J10.C18, J10.C20, J10.C21, J10.C23, J10.C24, J10.C26, J10.C27, J10.C29, J10.C30, J10.C32, J10.C33, J10.C36, J10.C38, J10.C40, J10.D02, J10.D03, J10.D04, J10.D05, J10.D06, J10.D07, J10.D08, J10.D09, J10.D10, J10.D11, J10.D12, J10.D13, J10.D14, J10.D15, J10.D16, J10.D17, J10.D18, J10.D19, J10.D20, J10.D21, J10.D22, J10.D23, J10.D24, J10.D25, J10.D26, J10.D27, J10.D28, J10.D29, J10.D30, J10.D31, J10.D32, J10.D33, J10.D35, J10.D37, J10.D39, J10.E02, J10.E03, J10.E04, J10.E05, J10.E06, J10.E07, J10.E08, J10.E09, J10.E10, J10.E11, J10.E12, J10.E13, J10.E14, J10.E15, J10.E16, J10.E17, J10.E18, J10.E19, J10.E20, J10.E21, J10.E22, J10.E23, J10.E24, J10.E25, J10.E26, J10.E27, J10.E28, J10.E29, J10.E30, J10.E31, J10.E32, J10.E33, J10.E36, J10.E38, J10.E40, J10.F01, J10.F02, J10.F03, J10.F04, J10.F06, J10.F07, J10.F09, J10.F10, J10.F12, J10.F13, J10.F15, J10.F16, J10.F18, J10.F19, J10.F21, J10.F22, J10.F24, J10.F25, J10.F27, J10.F28, J10.F30, J10.F31, J10.F33, J10.F34, J10.F35, J10.F37, J10.F39, J10.G03, J10.G04, J10.G06, J10.G07, J10.G09, J10.G10, J10.G12, J10.G13, J10.G15, J10.G16, J10.G18, J10.G19, J10.G21, J10.G22, J10.G24, J10.G25, J10.G27, J10.G28, J10.G30, J10.G31, J10.G33, J10.G34, J10.G36, J10.G38, J10.G40, J10.H03, J10.H04, J10.H05, J10.H06, J10.H07, J10.H08, J10.H09, J10.H10, J10.H11, J10.H12, J10.H13, J10.H14, J10.H15, J10.H16, J10.H17, J10.H18, J10.H19, J10.H20, J10.H21, J10.H22, J10.H23, J10.H24, J10.H25, J10.H26, J10.H27, J10.H28, J10.H29, J10.H30, J10.H31, J10.H32, J10.H33, J10.H35, J10.H37, J10.H39; no longer J10.A02, J10.A03, J10.A04, J10.A05, J10.A06, J10.A07, J10.A08, J10.A09, J10.A10, J10.A11, J10.A12, J10.A13, J10.A14, J10.A14, J10.A15, J10.A15, J10.A15, J10.A16, J10.A16, J10.A17, J10.A17, J10.A18, J10.A18, J10.A18, J10.A19, J10.A19, J10.A20, J10.A20, J10.A21, J10.A21, J10.A21, J10.A22, J10.A22, J10.A23, J10.A23, J10.A24, J10.A24, J10.A24, J10.A25, J10.A25, J10.A26, J10.A26, J10.A27, J10.A27, J10.A27, J10.A28, J10.A28, J10.A29, J10.A30, J10.A31, J10.A32, J10.A33, J10.B02, J10.B02, J10.B03, J10.B03, J10.B04, J10.B04, J10.B05, J10.B05, J10.B06, J10.B06, J10.B07, J10.B07, J10.B08, J10.B08, J10.B09, J10.B09, J10.B10, J10.B10, J10.B11, J10.B11, J10.B12, J10.B12, J10.B13, J10.B13, J10.B14, J10.B14, J10.B15, J10.B15, J10.B15, J10.B16, J10.B16, J10.B16, J10.B17, J10.B17, J10.B18, J10.B18, J10.B18, J10.B19, J10.B19, J10.B19, J10.B20, J10.B20, J10.B21, J10.B21, J10.B21, J10.B22, J10.B22, J10.B22, J10.B23, J10.B23, J10.B24, J10.B24, J10.B24, J10.B25, J10.B25, J10.B25, J10.B26, J10.B26, J10.B27, J10.B27, J10.B27, J10.B28, J10.B28, J10.B28, J10.B29, J10.B29, J10.B30, J10.B30, J10.B31, J10.B31, J10.B32, J10.B32, J10.B33, J10.B33
- net VCC12_SW: now reaches J10.A01
- net VCC12_SW: now also J10.B01, J10.C01, J10.D01, J10.E01
- net UTIL_3V3: now reaches J10.A34
- net UTIL_3V3: now also J10.B34, J10.C34, J10.D34, J10.E34, J10.H34
- net VCC1V8_BUS: now reaches J10.A35
- net VCC1V8_BUS: now also J10.C35
- net DACIO_00: now reaches J10.A37
- net DACIO_01: now reaches J10.A39
- net DAC_CLKIN_0_N: now reaches J10.B04
- net DAC_CLKIN_2_N: now reaches J10.B07
- net RFMC_DAC_00_N: now reaches J10.B10
- net RFMC_DAC_02_N: now reaches J10.B13
- net DACIO_02: now reaches J10.B36
- net DACIO_03: now reaches J10.B38
- net DACIO_04: now reaches J10.B40
- removed net DAC_C0_N: J10.A25
- net DAC_C0_P: no longer names the net of J10.B25
- removed net DAC_C1_N: J10.A26
- removed net DAC_C1_P: J10.B26
- removed net DAC_D0_N: J10.A22
- net DAC_D0_P: no longer names the net of J10.B22
- removed net DAC_D1_N: J10.A23
- removed net DAC_D1_P: J10.B23
- new net DACIO_05: J10.C37
- new net DACIO_06: J10.C39
- new net DACIO_07: J10.D36
- new net DACIO_08: J10.D38
- new net DACIO_09: J10.D40
- new net DACIO_10: J10.E37
- new net DACIO_11: J10.E39
- new net DACIO_12: J10.F36
- new net DACIO_13: J10.F38
- new net DACIO_14: J10.F40
- new net DACIO_15: J10.G37
- new net DACIO_16: J10.G39
- new net DACIO_17: J10.H36
- new net DACIO_18: J10.H38
- new net DACIO_19: J10.H40
- new net DAC_AVTT_BUS: J10.G01, J10.G02, J10.H01, J10.H02
- new net DAC_CLKIN_0_P: J10.C04
- new net DAC_CLKIN_1_N: J10.F05
- new net DAC_CLKIN_1_P: J10.G05
- new net DAC_CLKIN_2_P: J10.C07
- new net DAC_CLKIN_3_N: J10.F08
- new net DAC_CLKIN_3_P: J10.G08
- new net RFMC_DAC_00_P: J10.C10
- new net RFMC_DAC_01_N: J10.F11
- new net RFMC_DAC_01_P: J10.G11
- new net RFMC_DAC_02_P: J10.C13
- new net RFMC_DAC_03_N: J10.F14
- new net RFMC_DAC_03_P: J10.G14
- no-connect marks 0 -> 66
Other:
- moved on the sheet: J10B, J10C, J10D
