File: RFSoC_Frontend/RFSoC_Frontend.kicad_pcb (KiCad board)
At the start: 4 copper layers, 165.1 x 44.6 mm, 71 parts, among them J1 Conn_Coaxial, J10 LPAM-40-01.0-X-08-X-K-TR, J2 Conn_Coaxial, J3 Conn_Coaxial, J4 Conn_Coaxial, J5 Conn_Coaxial, J6 Conn_Coaxial, J7 Conn_Coaxial, J8 Conn_Coaxial, J9 LPAM-40-01.0-X-08-X-K-TR, U1 TCM2-33WX+, U2 TCM2-33WX+, U3 TCM2-33WX+, U4 TCM2-33WX+, U5 TCM2-33WX+, U6 TCM2-33WX+, U7 TCM2-33WX+, U8 TCM2-33WX+

Commit message: partial update of labels
Parts:
- moved C10 96.1 mm to (112.8, 89.0)
- moved C7 96.1 mm to (183.1, 89.0)
- moved C9 96.1 mm to (113.9, 89.0)
- moved R11 96.1 mm to (183.1, 85.4)
- moved R14 96.1 mm to (196.6, 87.5)
- moved R15 96.1 mm to (169.1, 86.9)
- moved R17 96.1 mm to (113.4, 87.2)
- moved R2 96.1 mm to (196.6, 83.9)
- moved R23 96.1 mm to (85.3, 85.3)
- moved R3 96.1 mm to (169.1, 83.4)
- moved R31 96.1 mm to (99.5, 83.6)
- moved U2 96.1 mm to (196.9, 93.2)
- moved U4 96.1 mm to (182.4, 92.8)
- moved U8 96.1 mm to (128.4, 92.6)
- moved C11 96.1 mm to (85.3, 88.9)
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Other:
- board text added: "1"
- board text added: "10"
- board text added: "15"
- board text added: "20"
- board text added: "25"
- board text added: "30"
- board text added: "35"
- board text added: "40"
- board text added: "5"
- board text added: "A"
- board text added: "ADC--- PAIR --,--"
- board text added: "ADC224 PAIR 0,1"
- board text added: "B"
- board text added: "B19"
- board text added: "B19,C19 RFMC_DAC_06"
- board text added: "C"
- board text added: "C19"
- board text added: "D"
- board text added: "DAC229 PAIR 0,1"
- board text added: "DAC229 PAIR 2,3"
- board text added: "E"
- board text added: "F"
- board text added: "F20"
- board text added: "F20,G20 RFMC_ADC_07"
- board text added: "G"
- board text added: "G20"
- board text added: "H"
- board text added: "RFMC ADC"
- board text added: "RFMC DAC"

Commit message: Finished Updated ADC schematic
ADC schematic was modified to match the pin map between
the rfsoc and the xm500.
Connections:
- net Net-(J9-PadA02) renamed /FMC BANK 0 (ADC)/ADCIO_00
- net Net-(J9-PadA04) renamed /FMC BANK 0 (ADC)/ADCIO_01
- net Net-(J9-PadA21) renamed /FMC BANK 0 (ADC)/VCM01_224
- net Net-(J9-PadB01) renamed /FMC BANK 0 (ADC)/ADCIO_02
- net Net-(J9-PadB03) renamed /FMC BANK 0 (ADC)/ADCIO_03
- net Net-(J9-PadB36) renamed /FMC BANK 0 (ADC)/ADC_CLKIN_0_N
- net Net-(J9-PadB39) renamed /FMC BANK 0 (ADC)/ADC_CLKIN_2_N
- net Net-(J9-PadC04) renamed /FMC BANK 0 (ADC)/ADCIO_06
- net Net-(J9-PadC36) renamed /FMC BANK 0 (ADC)/ADC_CLKIN_0_P
- net Net-(J9-PadC39) renamed /FMC BANK 0 (ADC)/ADC_CLKIN_2_P
- net Net-(J9-PadD01) renamed /FMC BANK 0 (ADC)/ADCIO_07
- net Net-(J9-PadD03) renamed /FMC BANK 0 (ADC)/ADCIO_08
- net Net-(J9-PadD05) renamed /FMC BANK 0 (ADC)/ADCIO_09
- net Net-(J9-PadD21) renamed /FMC BANK 0 (ADC)/VCM23_225
- net Net-(J9-PadE02) renamed /FMC BANK 0 (ADC)/ADCIO_10
- net Net-(J9-PadE04) renamed /FMC BANK 0 (ADC)/ADCIO_11
- net Net-(J9-PadE06) renamed /FMC BANK 0 (ADC)/RFMC_I2C_SDA
- net Net-(J9-PadE21) renamed /FMC BANK 0 (ADC)/VCM01_226
- net Net-(J9-PadF01) renamed /FMC BANK 0 (ADC)/ADCIO_12
- net Net-(J9-PadF03) renamed /FMC BANK 0 (ADC)/ADCIO_13
- net Net-(J9-PadF05) renamed /FMC BANK 0 (ADC)/ADCIO_14
- net Net-(J9-PadF21) renamed /FMC BANK 0 (ADC)/VCM23_226
- net Net-(J9-PadF35) renamed /FMC BANK 0 (ADC)/ADC_CLKIN_1_N
- net Net-(J9-PadF38) renamed /FMC BANK 0 (ADC)/ADC_CLKIN_3_N
- net Net-(J9-PadG02) renamed /FMC BANK 0 (ADC)/ADCIO_15
- net Net-(J9-PadG04) renamed /FMC BANK 0 (ADC)/ADCIO_16
- net Net-(J9-PadG06) renamed /FMC BANK 0 (ADC)/RFMC_I2C_SCL
- net Net-(J9-PadG21) renamed /FMC BANK 0 (ADC)/VCM01_227
- net Net-(J9-PadG35) renamed /FMC BANK 0 (ADC)/ADC_CLKIN_1_P
- net Net-(J9-PadG38) renamed /FMC BANK 0 (ADC)/ADC_CLKIN_3_P
- net Net-(J9-PadH01) renamed /FMC BANK 0 (ADC)/ADCIO_17
- net Net-(J9-PadH03) renamed /FMC BANK 0 (ADC)/ADCIO_18
- net Net-(J9-PadH05) renamed /FMC BANK 0 (ADC)/ADCIO_19
- net Net-(J9-PadH21) renamed /FMC BANK 0 (ADC)/VCM23_227
- J10 pad A01: Net-(J10-PadA01) -> unconnected-(J10-PadA01)
- J10 pad A34: Net-(J10-PadA34) -> unconnected-(J10-PadA34)
- J10 pad A35: Net-(J10-PadA35) -> unconnected-(J10-PadA35)
- J10 pad A36: Net-(J10-PadA36) -> unconnected-(J10-PadA36)
- J10 pad A37: Net-(J10-PadA37) -> unconnected-(J10-PadA37)
- J10 pad A38: Net-(J10-PadA38) -> unconnected-(J10-PadA38)
- J10 pad A39: Net-(J10-PadA39) -> unconnected-(J10-PadA39)
- J10 pad A40: Net-(J10-PadA40) -> unconnected-(J10-PadA40)
- J10 pad B01: Net-(J10-PadB01) -> unconnected-(J10-PadB01)
- J10 pad B02: Net-(J10-PadB02) -> unconnected-(J10-PadB02)
- J10 pad B03: Net-(J10-PadB03) -> unconnected-(J10-PadB03)
- J10 pad B04: Net-(J10-PadB04) -> unconnected-(J10-PadB04)
- J10 pad B05: Net-(J10-PadB05) -> unconnected-(J10-PadB05)
- J10 pad B06: Net-(J10-PadB06) -> unconnected-(J10-PadB06)
- J10 pad B07: Net-(J10-PadB07) -> unconnected-(J10-PadB07)
- J10 pad B08: Net-(J10-PadB08) -> unconnected-(J10-PadB08)
- J10 pad B09: Net-(J10-PadB09) -> unconnected-(J10-PadB09)
- J10 pad B10: Net-(J10-PadB10) -> unconnected-(J10-PadB10)
- J10 pad B11: Net-(J10-PadB11) -> unconnected-(J10-PadB11)
- J10 pad B12: Net-(J10-PadB12) -> unconnected-(J10-PadB12)
- J10 pad B13: Net-(J10-PadB13) -> unconnected-(J10-PadB13)
- J10 pad B28: Net-(J10-PadB28) -> unconnected-(J10-PadB28)
- J10 pad B29: Net-(J10-PadB29) -> unconnected-(J10-PadB29)
- J10 pad B30: Net-(J10-PadB30) -> unconnected-(J10-PadB30)
- J10 pad B31: Net-(J10-PadB31) -> unconnected-(J10-PadB31)
- J10 pad B32: Net-(J10-PadB32) -> unconnected-(J10-PadB32)
- J10 pad B33: Net-(J10-PadB33) -> unconnected-(J10-PadB33)
- J10 pad B34: Net-(J10-PadB34) -> unconnected-(J10-PadB34)
- J10 pad B35: Net-(J10-PadB35) -> unconnected-(J10-PadB35)
- J10 pad B36: Net-(J10-PadB36) -> unconnected-(J10-PadB36)
- J10 pad B37: Net-(J10-PadB37) -> unconnected-(J10-PadB37)
- J10 pad B38: Net-(J10-PadB38) -> unconnected-(J10-PadB38)
- J10 pad B39: Net-(J10-PadB39) -> unconnected-(J10-PadB39)
- J10 pad B40: Net-(J10-PadB40) -> unconnected-(J10-PadB40)
- J10 pad C01: Net-(J10-PadC01) -> unconnected-(J10-PadC01)
- J10 pad C02: Net-(J10-PadC02) -> unconnected-(J10-PadC02)
- J10 pad C03: Net-(J10-PadC03) -> unconnected-(J10-PadC03)
- J10 pad C04: Net-(J10-PadC04) -> unconnected-(J10-PadC04)
- J10 pad C05: Net-(J10-PadC05) -> unconnected-(J10-PadC05)
- J10 pad C06: Net-(J10-PadC06) -> unconnected-(J10-PadC06)
- J10 pad C07: Net-(J10-PadC07) -> unconnected-(J10-PadC07)
- J10 pad C08: Net-(J10-PadC08) -> unconnected-(J10-PadC08)
- J10 pad C09: Net-(J10-PadC09) -> unconnected-(J10-PadC09)
- J10 pad C10: Net-(J10-PadC10) -> unconnected-(J10-PadC10)
- J10 pad C11: Net-(J10-PadC11) -> unconnected-(J10-PadC11)
- J10 pad C12: Net-(J10-PadC12) -> unconnected-(J10-PadC12)
- J10 pad C13: Net-(J10-PadC13) -> unconnected-(J10-PadC13)
- J10 pad C28: Net-(J10-PadC28) -> unconnected-(J10-PadC28)
- J10 pad C29: Net-(J10-PadC29) -> unconnected-(J10-PadC29)
- J10 pad C30: Net-(J10-PadC30) -> unconnected-(J10-PadC30)
- J10 pad C31: Net-(J10-PadC31) -> unconnected-(J10-PadC31)
- J10 pad C32: Net-(J10-PadC32) -> unconnected-(J10-PadC32)
- J10 pad C33: Net-(J10-PadC33) -> unconnected-(J10-PadC33)
- J10 pad C34: Net-(J10-PadC34) -> unconnected-(J10-PadC34)
- J10 pad C35: Net-(J10-PadC35) -> unconnected-(J10-PadC35)
- J10 pad C36: Net-(J10-PadC36) -> unconnected-(J10-PadC36)
- J10 pad C37: Net-(J10-PadC37) -> unconnected-(J10-PadC37)
- J10 pad C38: Net-(J10-PadC38) -> unconnected-(J10-PadC38)
- J10 pad C39: Net-(J10-PadC39) -> unconnected-(J10-PadC39)
- J10 pad C40: Net-(J10-PadC40) -> unconnected-(J10-PadC40)
- J10 pad D01: Net-(J10-PadD01) -> unconnected-(J10-PadD01)
- J10 pad D34: Net-(J10-PadD34) -> unconnected-(J10-PadD34)
- J10 pad D35: Net-(J10-PadD35) -> unconnected-(J10-PadD35)
- J10 pad D36: Net-(J10-PadD36) -> unconnected-(J10-PadD36)
- J10 pad D37: Net-(J10-PadD37) -> unconnected-(J10-PadD37)
- J10 pad D38: Net-(J10-PadD38) -> unconnected-(J10-PadD38)
- J10 pad D39: Net-(J10-PadD39) -> unconnected-(J10-PadD39)
- J10 pad D40: Net-(J10-PadD40) -> unconnected-(J10-PadD40)
- J10 pad E01: Net-(J10-PadE01) -> unconnected-(J10-PadE01)
- J10 pad E34: Net-(J10-PadE34) -> unconnected-(J10-PadE34)
- J10 pad E35: Net-(J10-PadE35) -> unconnected-(J10-PadE35)
- J10 pad E36: Net-(J10-PadE36) -> unconnected-(J10-PadE36)
- J10 pad E37: Net-(J10-PadE37) -> unconnected-(J10-PadE37)
- J10 pad E38: Net-(J10-PadE38) -> unconnected-(J10-PadE38)
- J10 pad E39: Net-(J10-PadE39) -> unconnected-(J10-PadE39)
- J10 pad E40: Net-(J10-PadE40) -> unconnected-(J10-PadE40)
- J10 pad F01: Net-(J10-PadF01) -> unconnected-(J10-PadF01)
- J10 pad F02: Net-(J10-PadF02) -> unconnected-(J10-PadF02)
- J10 pad F03: Net-(J10-PadF03) -> unconnected-(J10-PadF03)
- J10 pad F04: Net-(J10-PadF04) -> unconnected-(J10-PadF04)
- J10 pad F05: Net-(J10-PadF05) -> unconnected-(J10-PadF05)
- J10 pad F06: Net-(J10-PadF06) -> unconnected-(J10-PadF06)
- J10 pad F07: Net-(J10-PadF07) -> unconnected-(J10-PadF07)
- J10 pad F08: Net-(J10-PadF08) -> unconnected-(J10-PadF08)
- J10 pad F09: Net-(J10-PadF09) -> unconnected-(J10-PadF09)
- J10 pad F10: Net-(J10-PadF10) -> unconnected-(J10-PadF10)
- J10 pad F11: Net-(J10-PadF11) -> unconnected-(J10-PadF11)
- J10 pad F12: Net-(J10-PadF12) -> unconnected-(J10-PadF12)
- J10 pad F13: Net-(J10-PadF13) -> unconnected-(J10-PadF13)
- J10 pad F14: Net-(J10-PadF14) -> unconnected-(J10-PadF14)
- J10 pad F29: Net-(J10-PadF29) -> unconnected-(J10-PadF29)
- J10 pad F30: Net-(J10-PadF30) -> unconnected-(J10-PadF30)
- J10 pad F31: Net-(J10-PadF31) -> unconnected-(J10-PadF31)
- J10 pad F32: Net-(J10-PadF32) -> unconnected-(J10-PadF32)
- J10 pad F33: Net-(J10-PadF33) -> unconnected-(J10-PadF33)
- J10 pad F34: Net-(J10-PadF34) -> unconnected-(J10-PadF34)
- J10 pad F35: Net-(J10-PadF35) -> unconnected-(J10-PadF35)
- J10 pad F36: Net-(J10-PadF36) -> unconnected-(J10-PadF36)
- J10 pad F37: Net-(J10-PadF37) -> unconnected-(J10-PadF37)
- J10 pad F38: Net-(J10-PadF38) -> unconnected-(J10-PadF38)
- J10 pad F39: Net-(J10-PadF39) -> unconnected-(J10-PadF39)
- J10 pad F40: Net-(J10-PadF40) -> unconnected-(J10-PadF40)
- J10 pad G01: Net-(J10-PadG01) -> unconnected-(J10-PadG01)
- J10 pad G02: Net-(J10-PadG02) -> unconnected-(J10-PadG02)
- J10 pad G03: Net-(J10-PadG03) -> unconnected-(J10-PadG03)
- J10 pad G04: Net-(J10-PadG04) -> unconnected-(J10-PadG04)
- J10 pad G05: Net-(J10-PadG05) -> unconnected-(J10-PadG05)
- J10 pad G06: Net-(J10-PadG06) -> unconnected-(J10-PadG06)
- J10 pad G07: Net-(J10-PadG07) -> unconnected-(J10-PadG07)
- J10 pad G08: Net-(J10-PadG08) -> unconnected-(J10-PadG08)
- J10 pad G09: Net-(J10-PadG09) -> unconnected-(J10-PadG09)
- J10 pad G10: Net-(J10-PadG10) -> unconnected-(J10-PadG10)
- J10 pad G11: Net-(J10-PadG11) -> unconnected-(J10-PadG11)
- J10 pad G12: Net-(J10-PadG12) -> unconnected-(J10-PadG12)
- J10 pad G13: Net-(J10-PadG13) -> unconnected-(J10-PadG13)
- J10 pad G14: Net-(J10-PadG14) -> unconnected-(J10-PadG14)
- J10 pad G29: Net-(J10-PadG29) -> unconnected-(J10-PadG29)
- J10 pad G30: Net-(J10-PadG30) -> unconnected-(J10-PadG30)
- J10 pad G31: Net-(J10-PadG31) -> unconnected-(J10-PadG31)
- J10 pad G32: Net-(J10-PadG32) -> unconnected-(J10-PadG32)
- J10 pad G33: Net-(J10-PadG33) -> unconnected-(J10-PadG33)
- J10 pad G34: Net-(J10-PadG34) -> unconnected-(J10-PadG34)
- J10 pad G35: Net-(J10-PadG35) -> unconnected-(J10-PadG35)
- J10 pad G36: Net-(J10-PadG36) -> unconnected-(J10-PadG36)
- J10 pad G37: Net-(J10-PadG37) -> unconnected-(J10-PadG37)
- J10 pad G38: Net-(J10-PadG38) -> unconnected-(J10-PadG38)
- J10 pad G39: Net-(J10-PadG39) -> unconnected-(J10-PadG39)
- J10 pad G40: Net-(J10-PadG40) -> unconnected-(J10-PadG40)
- J10 pad H01: Net-(J10-PadH01) -> unconnected-(J10-PadH01)
- J10 pad H34: Net-(J10-PadH34) -> unconnected-(J10-PadH34)
- J10 pad H35: Net-(J10-PadH35) -> unconnected-(J10-PadH35)
- J10 pad H36: Net-(J10-PadH36) -> unconnected-(J10-PadH36)
- J10 pad H37: Net-(J10-PadH37) -> unconnected-(J10-PadH37)
- J10 pad H38: Net-(J10-PadH38) -> unconnected-(J10-PadH38)
- J10 pad H39: Net-(J10-PadH39) -> unconnected-(J10-PadH39)
- J10 pad H40: Net-(J10-PadH40) -> unconnected-(J10-PadH40)
- J9 pad A01: Net-(J9-PadA01) -> GND
- J9 pad A03: Net-(J9-PadA03) -> GND
- J9 pad A05: Net-(J9-PadA05) -> GND
- J9 pad A06: Net-(J9-PadA06) -> /FMC BANK 0 (ADC)/VCC1V8_BUS
- J9 pad A07: Net-(J9-PadA07) -> /FMC BANK 0 (ADC)/UTIL_3V3
- J9 pad B02: Net-(J9-PadB02) -> GND
- J9 pad B04: Net-(J9-PadB04) -> GND
- J9 pad B05: Net-(J9-PadB05) -> /FMC BANK 0 (ADC)/ADCIO_05
- J9 pad B06: Net-(J9-PadB06) -> GND
- J9 pad B07: Net-(J9-PadB07) -> GND
- J9 pad B21: GND -> /FMC BANK 0 (ADC)/VCM23_224
- J9 pad B22: Net-(J9-PadB22) -> GND
- J9 pad B23: Net-(J9-PadB23) -> GND
- J9 pad B24: Net-(J9-PadB24) -> unconnected-(J9-PadB24)
- J9 pad B25: Net-(J9-PadB25) -> GND
- J9 pad B26: Net-(J9-PadB26) -> GND
- J9 pad B27: Net-(J9-PadB27) -> unconnected-(J9-PadB27)
- J9 pad B28: Net-(J9-PadB28) -> GND
- J9 pad B29: Net-(J9-PadB29) -> GND
- J9 pad B30: Net-(J9-PadB30) -> unconnected-(J9-PadB30)
- J9 pad B31: Net-(J9-PadB31) -> GND
- J9 pad B32: Net-(J9-PadB32) -> GND
- J9 pad B33: Net-(J9-PadB33) -> unconnected-(J9-PadB33)
- J9 pad B34: Net-(J9-PadB34) -> GND
- J9 pad B35: Net-(J9-PadB35) -> GND
- J9 pad B37: Net-(J9-PadB37) -> GND
- J9 pad B38: Net-(J9-PadB38) -> GND
- J9 pad B40: Net-(J9-PadB40) -> GND
- J9 pad C01: Net-(J9-PadC01) -> GND
- J9 pad C02: Net-(J9-PadC02) -> /FMC BANK 0 (ADC)/ADCIO_05
- J9 pad C03: Net-(J9-PadC03) -> GND
- J9 pad C05: Net-(J9-PadC05) -> GND
- J9 pad C06: Net-(J9-PadC06) -> /FMC BANK 0 (ADC)/VCC1V8_BUS
- J9 pad C07: Net-(J9-PadC07) -> /FMC BANK 0 (ADC)/UTIL_3V3
- J9 pad C21: GND -> /FMC BANK 0 (ADC)/VCM01_225
- J9 pad C22: Net-(J9-PadC22) -> GND
- J9 pad C23: Net-(J9-PadC23) -> GND
- J9 pad C24: Net-(J9-PadC24) -> unconnected-(J9-PadC24)
- J9 pad C25: Net-(J9-PadC25) -> GND
- J9 pad C26: Net-(J9-PadC26) -> GND
- J9 pad C27: Net-(J9-PadC27) -> unconnected-(J9-PadC27)
- J9 pad C28: Net-(J9-PadC28) -> GND
- J9 pad C29: Net-(J9-PadC29) -> GND
- J9 pad C30: Net-(J9-PadC30) -> unconnected-(J9-PadC30)
- J9 pad C31: Net-(J9-PadC31) -> GND
- J9 pad C32: Net-(J9-PadC32) -> GND
- J9 pad C33: Net-(J9-PadC33) -> unconnected-(J9-PadC33)
- J9 pad C34: Net-(J9-PadC34) -> GND
- J9 pad C35: Net-(J9-PadC35) -> GND
- J9 pad C37: Net-(J9-PadC37) -> GND
- J9 pad C38: Net-(J9-PadC38) -> GND
- J9 pad C40: Net-(J9-PadC40) -> GND
- J9 pad D02: Net-(J9-PadD02) -> GND
- J9 pad D04: Net-(J9-PadD04) -> GND
- J9 pad D06: Net-(J9-PadD06) -> GND
- J9 pad D07: Net-(J9-PadD07) -> /FMC BANK 0 (ADC)/UTIL_3V3
- J9 pad E01: Net-(J9-PadE01) -> GND
- J9 pad E03: Net-(J9-PadE03) -> GND
- J9 pad E05: Net-(J9-PadE05) -> GND
- J9 pad E07: Net-(J9-PadE07) -> /FMC BANK 0 (ADC)/UTIL_3V3
- J9 pad F02: Net-(J9-PadF02) -> GND
- J9 pad F04: Net-(J9-PadF04) -> GND
- J9 pad F06: Net-(J9-PadF06) -> GND
- J9 pad F07: Net-(J9-PadF07) -> /FMC BANK 0 (ADC)/UTIL_3V3
- J9 pad F22: Net-(J9-PadF22) -> GND
- J9 pad F23: Net-(J9-PadF23) -> unconnected-(J9-PadF23)
- J9 pad F24: Net-(J9-PadF24) -> GND
- J9 pad F25: Net-(J9-PadF25) -> GND
- J9 pad F26: Net-(J9-PadF26) -> unconnected-(J9-PadF26)
- J9 pad F27: Net-(J9-PadF27) -> GND
- J9 pad F28: Net-(J9-PadF28) -> GND
- J9 pad F29: Net-(J9-PadF29) -> unconnected-(J9-PadF29)
- J9 pad F30: Net-(J9-PadF30) -> GND
- J9 pad F31: Net-(J9-PadF31) -> GND
- J9 pad F32: Net-(J9-PadF32) -> unconnected-(J9-PadF32)
- J9 pad F33: Net-(J9-PadF33) -> GND
- J9 pad F34: Net-(J9-PadF34) -> GND
- J9 pad F36: Net-(J9-PadF36) -> GND
- J9 pad F37: Net-(J9-PadF37) -> GND
- J9 pad F39: Net-(J9-PadF39) -> GND
- J9 pad F40: Net-(J9-PadF40) -> GND
- J9 pad G01: Net-(J9-PadG01) -> GND
- J9 pad G03: Net-(J9-PadG03) -> GND
- J9 pad G05: Net-(J9-PadG05) -> GND
- J9 pad G07: Net-(J9-PadG07) -> /FMC BANK 0 (ADC)/UTIL_3V3
- J9 pad G22: Net-(J9-PadG22) -> GND
- J9 pad G23: Net-(J9-PadG23) -> unconnected-(J9-PadG23)
- J9 pad G24: Net-(J9-PadG24) -> GND
- J9 pad G25: Net-(J9-PadG25) -> GND
- J9 pad G26: Net-(J9-PadG26) -> unconnected-(J9-PadG26)
- J9 pad G27: Net-(J9-PadG27) -> GND
- J9 pad G28: Net-(J9-PadG28) -> GND
- J9 pad G29: Net-(J9-PadG29) -> unconnected-(J9-PadG29)
- J9 pad G30: Net-(J9-PadG30) -> GND
- J9 pad G31: Net-(J9-PadG31) -> GND
- J9 pad G32: Net-(J9-PadG32) -> unconnected-(J9-PadG32)
- J9 pad G33: Net-(J9-PadG33) -> GND
- J9 pad G34: Net-(J9-PadG34) -> GND
- J9 pad G36: Net-(J9-PadG36) -> GND
- J9 pad G37: Net-(J9-PadG37) -> GND
- J9 pad G39: Net-(J9-PadG39) -> GND
- J9 pad G40: Net-(J9-PadG40) -> GND
- J9 pad H02: Net-(J9-PadH02) -> GND
- J9 pad H04: Net-(J9-PadH04) -> GND
- J9 pad H06: Net-(J9-PadH06) -> GND
- J9 pad H07: Net-(J9-PadH07) -> /FMC BANK 0 (ADC)/UTIL_3V3
- U1 pad 1: Net-(U1-Pad1) -> unconnected-(U1-Pad1)
- U2 pad 1: Net-(U2-Pad1) -> unconnected-(U2-Pad1)
- U3 pad 1: Net-(U3-Pad1) -> unconnected-(U3-Pad1)
- U4 pad 1: Net-(U4-Pad1) -> unconnected-(U4-Pad1)
- U5 pad 1: Net-(U5-Pad1) -> unconnected-(U5-Pad1)
- U6 pad 1: Net-(U6-Pad1) -> unconnected-(U6-Pad1)
- U7 pad 1: Net-(U7-Pad1) -> unconnected-(U7-Pad1)
- U8 pad 1: Net-(U8-Pad1) -> unconnected-(U8-Pad1)

Commit message: updated all
Connections:
- J10 pad A01: unconnected-(J10-PadA01) -> /FMC BANK 1 (DAC)/VCC12_SW
- J10 pad A34: unconnected-(J10-PadA34) -> /FMC BANK 1 (DAC)/UTIL_3V3
- J10 pad A35: unconnected-(J10-PadA35) -> /FMC BANK 1 (DAC)/VCC1V8_BUS
- J10 pad A36: unconnected-(J10-PadA36) -> GND
- J10 pad A37: unconnected-(J10-PadA37) -> /FMC BANK 1 (DAC)/DACIO_00
- J10 pad A38: unconnected-(J10-PadA38) -> GND
- J10 pad A39: unconnected-(J10-PadA39) -> /FMC BANK 1 (DAC)/DACIO_01
- J10 pad A40: unconnected-(J10-PadA40) -> GND
- J10 pad B01: unconnected-(J10-PadB01) -> /FMC BANK 1 (DAC)/VCC12_SW
- J10 pad B02: unconnected-(J10-PadB02) -> GND
- J10 pad B03: unconnected-(J10-PadB03) -> GND
- J10 pad B04: unconnected-(J10-PadB04) -> /FMC BANK 1 (DAC)/DAC_CLKIN_0_N
- J10 pad B05: unconnected-(J10-PadB05) -> GND
- J10 pad B06: unconnected-(J10-PadB06) -> GND
- J10 pad B07: unconnected-(J10-PadB07) -> /FMC BANK 1 (DAC)/DAC_CLKIN_2_N
- J10 pad B08: unconnected-(J10-PadB08) -> GND
- J10 pad B09: unconnected-(J10-PadB09) -> GND
- J10 pad B10: unconnected-(J10-PadB10) -> /FMC BANK 1 (DAC)/RFMC_DAC_00_N
- J10 pad B11: unconnected-(J10-PadB11) -> GND
- J10 pad B12: unconnected-(J10-PadB12) -> GND
- J10 pad B13: unconnected-(J10-PadB13) -> /FMC BANK 1 (DAC)/RFMC_DAC_02_N
- J10 pad B22: DAC_D0_P -> unconnected-(J10-PadB22)
- J10 pad B25: DAC_C0_P -> unconnected-(J10-PadB25)
- J10 pad B29: unconnected-(J10-PadB29) -> GND
- J10 pad B30: unconnected-(J10-PadB30) -> GND
- J10 pad B32: unconnected-(J10-PadB32) -> GND
- J10 pad B33: unconnected-(J10-PadB33) -> GND
- J10 pad B34: unconnected-(J10-PadB34) -> /FMC BANK 1 (DAC)/UTIL_3V3
- J10 pad B35: unconnected-(J10-PadB35) -> GND
- J10 pad B36: unconnected-(J10-PadB36) -> /FMC BANK 1 (DAC)/DACIO_02
- J10 pad B37: unconnected-(J10-PadB37) -> GND
- J10 pad B38: unconnected-(J10-PadB38) -> /FMC BANK 1 (DAC)/DACIO_03
- J10 pad B39: unconnected-(J10-PadB39) -> GND
- J10 pad B40: unconnected-(J10-PadB40) -> /FMC BANK 1 (DAC)/DACIO_04
- J10 pad C01: unconnected-(J10-PadC01) -> /FMC BANK 1 (DAC)/VCC12_SW
- J10 pad C02: unconnected-(J10-PadC02) -> GND
- J10 pad C03: unconnected-(J10-PadC03) -> GND
- J10 pad C04: unconnected-(J10-PadC04) -> /FMC BANK 1 (DAC)/DAC_CLKIN_0_P
- J10 pad C05: unconnected-(J10-PadC05) -> GND
- J10 pad C06: unconnected-(J10-PadC06) -> GND
- J10 pad C07: unconnected-(J10-PadC07) -> /FMC BANK 1 (DAC)/DAC_CLKIN_2_P
- J10 pad C08: unconnected-(J10-PadC08) -> GND
- J10 pad C09: unconnected-(J10-PadC09) -> GND
- J10 pad C10: unconnected-(J10-PadC10) -> /FMC BANK 1 (DAC)/RFMC_DAC_00_P
- J10 pad C11: unconnected-(J10-PadC11) -> GND
- J10 pad C12: unconnected-(J10-PadC12) -> GND
- J10 pad C13: unconnected-(J10-PadC13) -> /FMC BANK 1 (DAC)/RFMC_DAC_02_P
- J10 pad C22: DAC_D0_N -> unconnected-(J10-PadC22)
- J10 pad C25: DAC_C0_N -> unconnected-(J10-PadC25)
- J10 pad C29: unconnected-(J10-PadC29) -> GND
- J10 pad C30: unconnected-(J10-PadC30) -> GND
- J10 pad C32: unconnected-(J10-PadC32) -> GND
- J10 pad C33: unconnected-(J10-PadC33) -> GND
- J10 pad C34: unconnected-(J10-PadC34) -> /FMC BANK 1 (DAC)/UTIL_3V3
- J10 pad C35: unconnected-(J10-PadC35) -> /FMC BANK 1 (DAC)/VCC1V8_BUS
- J10 pad C36: unconnected-(J10-PadC36) -> GND
- J10 pad C37: unconnected-(J10-PadC37) -> /FMC BANK 1 (DAC)/DACIO_05
- J10 pad C38: unconnected-(J10-PadC38) -> GND
- J10 pad C39: unconnected-(J10-PadC39) -> /FMC BANK 1 (DAC)/DACIO_06
- J10 pad C40: unconnected-(J10-PadC40) -> GND
- J10 pad D01: unconnected-(J10-PadD01) -> /FMC BANK 1 (DAC)/VCC12_SW
- J10 pad D34: unconnected-(J10-PadD34) -> /FMC BANK 1 (DAC)/UTIL_3V3
- J10 pad D35: unconnected-(J10-PadD35) -> GND
- J10 pad D36: unconnected-(J10-PadD36) -> /FMC BANK 1 (DAC)/DACIO_07
- J10 pad D37: unconnected-(J10-PadD37) -> GND
- J10 pad D38: unconnected-(J10-PadD38) -> /FMC BANK 1 (DAC)/DACIO_08
- J10 pad D39: unconnected-(J10-PadD39) -> GND
- J10 pad D40: unconnected-(J10-PadD40) -> /FMC BANK 1 (DAC)/DACIO_09
- J10 pad E01: unconnected-(J10-PadE01) -> /FMC BANK 1 (DAC)/VCC12_SW
- J10 pad E34: unconnected-(J10-PadE34) -> /FMC BANK 1 (DAC)/UTIL_3V3
- J10 pad E36: unconnected-(J10-PadE36) -> GND
- J10 pad E37: unconnected-(J10-PadE37) -> /FMC BANK 1 (DAC)/DACIO_10
- J10 pad E38: unconnected-(J10-PadE38) -> GND
- J10 pad E39: unconnected-(J10-PadE39) -> /FMC BANK 1 (DAC)/DACIO_11
- J10 pad E40: unconnected-(J10-PadE40) -> GND
- J10 pad F01: unconnected-(J10-PadF01) -> GND
- J10 pad F02: unconnected-(J10-PadF02) -> GND
- J10 pad F03: unconnected-(J10-PadF03) -> GND
- J10 pad F04: unconnected-(J10-PadF04) -> GND
- J10 pad F05: unconnected-(J10-PadF05) -> /FMC BANK 1 (DAC)/DAC_CLKIN_1_N
- J10 pad F06: unconnected-(J10-PadF06) -> GND
- J10 pad F07: unconnected-(J10-PadF07) -> GND
- J10 pad F08: unconnected-(J10-PadF08) -> /FMC BANK 1 (DAC)/DAC_CLKIN_3_N
- J10 pad F09: unconnected-(J10-PadF09) -> GND
- J10 pad F10: unconnected-(J10-PadF10) -> GND
- J10 pad F11: unconnected-(J10-PadF11) -> /FMC BANK 1 (DAC)/RFMC_DAC_01_N
- J10 pad F12: unconnected-(J10-PadF12) -> GND
- J10 pad F13: unconnected-(J10-PadF13) -> GND
- J10 pad F14: unconnected-(J10-PadF14) -> /FMC BANK 1 (DAC)/RFMC_DAC_03_N
- J10 pad F23: DAC_D1_P -> unconnected-(J10-PadF23)
- J10 pad F26: DAC_C1_P -> unconnected-(J10-PadF26)
- J10 pad F30: unconnected-(J10-PadF30) -> GND
- J10 pad F31: unconnected-(J10-PadF31) -> GND
- J10 pad F33: unconnected-(J10-PadF33) -> GND
- J10 pad F34: unconnected-(J10-PadF34) -> GND
- J10 pad F35: unconnected-(J10-PadF35) -> GND
- J10 pad F36: unconnected-(J10-PadF36) -> /FMC BANK 1 (DAC)/DACIO_12
- J10 pad F37: unconnected-(J10-PadF37) -> GND
- J10 pad F38: unconnected-(J10-PadF38) -> /FMC BANK 1 (DAC)/DACIO_13
- J10 pad F39: unconnected-(J10-PadF39) -> GND
- J10 pad F40: unconnected-(J10-PadF40) -> /FMC BANK 1 (DAC)/DACIO_14
- J10 pad G01: unconnected-(J10-PadG01) -> /FMC BANK 1 (DAC)/DAC_AVTT_BUS
- J10 pad G02: unconnected-(J10-PadG02) -> /FMC BANK 1 (DAC)/DAC_AVTT_BUS
- J10 pad G03: unconnected-(J10-PadG03) -> GND
- J10 pad G04: unconnected-(J10-PadG04) -> GND
- J10 pad G05: unconnected-(J10-PadG05) -> /FMC BANK 1 (DAC)/DAC_CLKIN_1_P
- J10 pad G06: unconnected-(J10-PadG06) -> GND
- J10 pad G07: unconnected-(J10-PadG07) -> GND
- J10 pad G08: unconnected-(J10-PadG08) -> /FMC BANK 1 (DAC)/DAC_CLKIN_3_P
- J10 pad G09: unconnected-(J10-PadG09) -> GND
- J10 pad G10: unconnected-(J10-PadG10) -> GND
- J10 pad G11: unconnected-(J10-PadG11) -> /FMC BANK 1 (DAC)/RFMC_DAC_01_P
- J10 pad G12: unconnected-(J10-PadG12) -> GND
- J10 pad G13: unconnected-(J10-PadG13) -> GND
- J10 pad G14: unconnected-(J10-PadG14) -> /FMC BANK 1 (DAC)/RFMC_DAC_03_P
- J10 pad G23: DAC_D1_N -> unconnected-(J10-PadG23)
- J10 pad G26: DAC_C1_N -> unconnected-(J10-PadG26)
- J10 pad G30: unconnected-(J10-PadG30) -> GND
- J10 pad G31: unconnected-(J10-PadG31) -> GND
- J10 pad G33: unconnected-(J10-PadG33) -> GND
- J10 pad G34: unconnected-(J10-PadG34) -> GND
- J10 pad G36: unconnected-(J10-PadG36) -> GND
- J10 pad G37: unconnected-(J10-PadG37) -> /FMC BANK 1 (DAC)/DACIO_15
- J10 pad G38: unconnected-(J10-PadG38) -> GND
- J10 pad G39: unconnected-(J10-PadG39) -> /FMC BANK 1 (DAC)/DACIO_16
- J10 pad G40: unconnected-(J10-PadG40) -> GND
- J10 pad H01: unconnected-(J10-PadH01) -> /FMC BANK 1 (DAC)/DAC_AVTT_BUS
- J10 pad H02: GND -> /FMC BANK 1 (DAC)/DAC_AVTT_BUS
- J10 pad H34: unconnected-(J10-PadH34) -> /FMC BANK 1 (DAC)/UTIL_3V3
- J10 pad H35: unconnected-(J10-PadH35) -> GND
- J10 pad H36: unconnected-(J10-PadH36) -> /FMC BANK 1 (DAC)/DACIO_17
- J10 pad H37: unconnected-(J10-PadH37) -> GND
- J10 pad H38: unconnected-(J10-PadH38) -> /FMC BANK 1 (DAC)/DACIO_18
- J10 pad H39: unconnected-(J10-PadH39) -> GND
- J10 pad H40: unconnected-(J10-PadH40) -> /FMC BANK 1 (DAC)/DACIO_19

Commit message: fork em
Parts:
- added G***: LOGO, LOGO, F.Cu at (63.3, 99.1)
Other:
- outline, holes or cut-outs redrawn
- board text added: "B10"
- board text added: "B13"
- board text added: "B16"
- board text added: "C10"
- board text added: "C13"
- board text added: "C16"
- board text added: "F09"
- board text added: "F12"
- board text added: "F17"
- board text added: "FORK 'EM"
- board text added: "G09"
- board text added: "G12"
- board text added: "G17"
- board text added: "Ryan Stephenson Cody Roberson Eric Weeks Arizona State University"

Commit message: updated silkscreens, degin DRC corrections
Parts:
- moved U1 0.30 mm to (211.6, 92.9)
- moved U2 0.28 mm to (196.9, 92.9)
Routing:
- net Net-(J2-Pad1): track 6.67 -> 7.36 mm
- net DAC_B1_P: track 31.6 -> 30.9 mm, vias 2 -> 1
- net Net-(J1-Pad1): track 6.73 -> 7.36 mm
- net DAC_B0_P: track 13.6 -> 13.3 mm, vias 2 -> 1
- net ADC_A0_P: vias 2 -> 1
- net ADC_A0_N: vias 2 -> 1
- net GND: vias 0 -> 78
- net DAC_B1_N: vias 2 -> 1
- net DAC_B0_N: vias 2 -> 1
- net DAC_A1_P: vias 2 -> 1
- net DAC_A1_N: vias 2 -> 1
- net DAC_A0_P: vias 2 -> 1
- net DAC_A0_N: vias 2 -> 1
- net ADC_B1_P: vias 2 -> 1
- net ADC_B1_N: vias 2 -> 1
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Other:
- outline, holes or cut-outs redrawn
- board text added: "ADC224 PAIR 0,1 (CHANNEL 0 I/Q)"
- board text added: "ADC225 PAIR 0,1 (CHANNEL 1 I/Q)"
- board text added: "DAC229 PAIR 0,1 (CHANNEL 1 I/Q)"
- board text added: "DAC229 PAIR 2,3 (CHANNEL 0 I/Q)"
- board text removed: "ADC--- PAIR --,--"
- board text removed: "ADC224 PAIR 0,1"
- board text removed: "DAC229 PAIR 0,1"
- board text removed: "DAC229 PAIR 2,3"
