File: RFSoC_Frontend/RFSoC_Frontend.kicad_pcb (KiCad board)
At the start: 4 copper layers, 165.1 x 44.6 mm, 71 parts, among them J1 Conn_Coaxial, J10 LPAM-40-01.0-X-08-X-K-TR, J2 Conn_Coaxial, J3 Conn_Coaxial, J4 Conn_Coaxial, J5 Conn_Coaxial, J6 Conn_Coaxial, J7 Conn_Coaxial, J8 Conn_Coaxial, J9 LPAM-40-01.0-X-08-X-K-TR, U1 TCM2-33WX+, U2 TCM2-33WX+, U3 TCM2-33WX+, U4 TCM2-33WX+, U5 TCM2-33WX+, U6 TCM2-33WX+, U7 TCM2-33WX+, U8 TCM2-33WX+

Commit message: Squashed commit of the following:
commit 11c362fd04afcdda8fc54016fc262973d8ee90dd
Author: cody <you@example.com>
Date:   Sat May 14 20:18:42 2022 -0700

    updated silkscreens, degin DRC corrections

commit c03c76887280f84603892cf274eefb7fb13b0fa8
Author: cody <you@example.com>
Date:   Fri May 13 16:10:57 2022 -0700

    fork em

commit e1673cb11a9ebe940ceda00a5b2ec080c415b465
Author: cody <you@example.com>
Date:   Fri May 13 15:38:00 2022 -0700

    updated all

commit 84fbdba19d4f5d8a85804f2c5d387b833a8e7f5e
Author: Cody Roberson <carobers@asu.edu>
Date:   Mon May 9 16:15:14 2022 -0700

    Finished Updated ADC schematic

    ADC schematic was modified to match the pin map between
    the rfsoc and the xm500.

commit 1e4de3bc2e504d4b0d3d294a2c6c5a2a5a485041
Author: cody <you@example.com>
Date:   Mon May 9 10:21:30 2022 -0700

    progress check

    Started Labeling process

commit 6cadb2acb3bb1a794e84b73e4dfc828af985fa6c
Author: cody <you@example.com>
Date:   Thu May 5 15:24:15 2022 -0700

    partial update of labels

commit 2dab10b1dfa9c61606f5d562ab6e543ae0948647
Merge: 76ba8d6 79e9342
Author: Cody Roberson <codyaroberson@outlook.com>
Date:   Wed Mar 9 20:07:10 2022 -0700

    Merge pull request #1 from CodyRoberson/twochannel_clk

    Twochannel clk

commit 79e93425439f23e00c2b0d92e892590d87fe78f7
Author: Cody Roberson <carobers@asu.edu>
Date:   Wed Mar 9 20:04:09 2022 -0700

    moved forkem and labeled ports

commit 9a4b6dc66818e11f3bb9969be501559d1f9e476d
Author: Cody Roberson <carobers@asu.edu>
Date:   Wed Mar 9 16:28:24 2022 -0700

    improvements

    Made improvement to kicad symbol and replaced footprint for baluns. They
    were incorrectly orientated with regards to pin numbering

commit 8d29e46f6a613ffa86cae2f2a7a070122b97e7eb
Author: Cody Roberson <carobers@asu.edu>
Date:   Wed Mar 9 14:50:01 2022 -0700

    added kicad symbol+footprint

commit 3c7e1566d05959f7dad261469b2e27b92f79ed87
Author: Cody Roberson <carobers@asu.edu>
Date:   Wed Mar 9 14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
Parts:
- added G***: LOGO, LOGO, F.Cu at (63.3, 99.1)
- moved C10 96.1 mm to (112.8, 89.0)
- moved C7 96.1 mm to (183.1, 89.0)
- moved C9 96.1 mm to (113.9, 89.0)
- moved R11 96.1 mm to (183.1, 85.4)
- moved R14 96.1 mm to (196.6, 87.5)
- moved R15 96.1 mm to (169.1, 86.9)
- moved R17 96.1 mm to (113.4, 87.2)
- moved R2 96.1 mm to (196.6, 83.9)
- moved R23 96.1 mm to (85.3, 85.3)
- moved R3 96.1 mm to (169.1, 83.4)
- moved R31 96.1 mm to (99.5, 83.6)
- moved U4 96.1 mm to (182.4, 92.8)
- moved U8 96.1 mm to (128.4, 92.6)
- moved C11 96.1 mm to (85.3, 88.9)
- moved C12 96.1 mm to (84.3, 88.9)
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Connections:
- net Net-(J10-PadA37) renamed /FMC BANK 1 (DAC)/DACIO_00
- net Net-(J10-PadA39) renamed /FMC BANK 1 (DAC)/DACIO_01
- net Net-(J10-PadB04) renamed /FMC BANK 1 (DAC)/DAC_CLKIN_0_N
- net Net-(J10-PadB07) renamed /FMC BANK 1 (DAC)/DAC_CLKIN_2_N
- net Net-(J10-PadB10) renamed /FMC BANK 1 (DAC)/RFMC_DAC_00_N
- net Net-(J10-PadB13) renamed /FMC BANK 1 (DAC)/RFMC_DAC_02_N
- net Net-(J10-PadB36) renamed /FMC BANK 1 (DAC)/DACIO_02
- net Net-(J10-PadB38) renamed /FMC BANK 1 (DAC)/DACIO_03
- net Net-(J10-PadB40) renamed /FMC BANK 1 (DAC)/DACIO_04
- net Net-(J10-PadC04) renamed /FMC BANK 1 (DAC)/DAC_CLKIN_0_P
- net Net-(J10-PadC07) renamed /FMC BANK 1 (DAC)/DAC_CLKIN_2_P
- net Net-(J10-PadC10) renamed /FMC BANK 1 (DAC)/RFMC_DAC_00_P
- net Net-(J10-PadC13) renamed /FMC BANK 1 (DAC)/RFMC_DAC_02_P
- net Net-(J10-PadC37) renamed /FMC BANK 1 (DAC)/DACIO_05
- net Net-(J10-PadC39) renamed /FMC BANK 1 (DAC)/DACIO_06
- net Net-(J10-PadD36) renamed /FMC BANK 1 (DAC)/DACIO_07
- net Net-(J10-PadD38) renamed /FMC BANK 1 (DAC)/DACIO_08
- net Net-(J10-PadD40) renamed /FMC BANK 1 (DAC)/DACIO_09
- net Net-(J10-PadE37) renamed /FMC BANK 1 (DAC)/DACIO_10
- net Net-(J10-PadE39) renamed /FMC BANK 1 (DAC)/DACIO_11
- net Net-(J10-PadF05) renamed /FMC BANK 1 (DAC)/DAC_CLKIN_1_N
- net Net-(J10-PadF08) renamed /FMC BANK 1 (DAC)/DAC_CLKIN_3_N
- net Net-(J10-PadF11) renamed /FMC BANK 1 (DAC)/RFMC_DAC_01_N
- net Net-(J10-PadF14) renamed /FMC BANK 1 (DAC)/RFMC_DAC_03_N
- net Net-(J10-PadF36) renamed /FMC BANK 1 (DAC)/DACIO_12
- net Net-(J10-PadF38) renamed /FMC BANK 1 (DAC)/DACIO_13
- net Net-(J10-PadF40) renamed /FMC BANK 1 (DAC)/DACIO_14
- net Net-(J10-PadG05) renamed /FMC BANK 1 (DAC)/DAC_CLKIN_1_P
- net Net-(J10-PadG08) renamed /FMC BANK 1 (DAC)/DAC_CLKIN_3_P
- net Net-(J10-PadG11) renamed /FMC BANK 1 (DAC)/RFMC_DAC_01_P
- net Net-(J10-PadG14) renamed /FMC BANK 1 (DAC)/RFMC_DAC_03_P
- net Net-(J10-PadG37) renamed /FMC BANK 1 (DAC)/DACIO_15
- net Net-(J10-PadG39) renamed /FMC BANK 1 (DAC)/DACIO_16
- net Net-(J10-PadH36) renamed /FMC BANK 1 (DAC)/DACIO_17
- net Net-(J10-PadH38) renamed /FMC BANK 1 (DAC)/DACIO_18
- net Net-(J10-PadH40) renamed /FMC BANK 1 (DAC)/DACIO_19
- net Net-(J9-PadA02) renamed /FMC BANK 0 (ADC)/ADCIO_00
- net Net-(J9-PadA04) renamed /FMC BANK 0 (ADC)/ADCIO_01
- net Net-(J9-PadA21) renamed /FMC BANK 0 (ADC)/VCM01_224
- net Net-(J9-PadB01) renamed /FMC BANK 0 (ADC)/ADCIO_02
- net Net-(J9-PadB03) renamed /FMC BANK 0 (ADC)/ADCIO_03
- net Net-(J9-PadB36) renamed /FMC BANK 0 (ADC)/ADC_CLKIN_0_N
- net Net-(J9-PadB39) renamed /FMC BANK 0 (ADC)/ADC_CLKIN_2_N
- net Net-(J9-PadC04) renamed /FMC BANK 0 (ADC)/ADCIO_06
- net Net-(J9-PadC36) renamed /FMC BANK 0 (ADC)/ADC_CLKIN_0_P
- net Net-(J9-PadC39) renamed /FMC BANK 0 (ADC)/ADC_CLKIN_2_P
- net Net-(J9-PadD01) renamed /FMC BANK 0 (ADC)/ADCIO_07
- net Net-(J9-PadD03) renamed /FMC BANK 0 (ADC)/ADCIO_08
- net Net-(J9-PadD05) renamed /FMC BANK 0 (ADC)/ADCIO_09
- net Net-(J9-PadD21) renamed /FMC BANK 0 (ADC)/VCM23_225
- net Net-(J9-PadE02) renamed /FMC BANK 0 (ADC)/ADCIO_10
- net Net-(J9-PadE04) renamed /FMC BANK 0 (ADC)/ADCIO_11
- net Net-(J9-PadE06) renamed /FMC BANK 0 (ADC)/RFMC_I2C_SDA
- net Net-(J9-PadE21) renamed /FMC BANK 0 (ADC)/VCM01_226
- net Net-(J9-PadF01) renamed /FMC BANK 0 (ADC)/ADCIO_12
- net Net-(J9-PadF03) renamed /FMC BANK 0 (ADC)/ADCIO_13
- net Net-(J9-PadF05) renamed /FMC BANK 0 (ADC)/ADCIO_14
- net Net-(J9-PadF21) renamed /FMC BANK 0 (ADC)/VCM23_226
- net Net-(J9-PadF35) renamed /FMC BANK 0 (ADC)/ADC_CLKIN_1_N
- net Net-(J9-PadF38) renamed /FMC BANK 0 (ADC)/ADC_CLKIN_3_N
- net Net-(J9-PadG02) renamed /FMC BANK 0 (ADC)/ADCIO_15
- net Net-(J9-PadG04) renamed /FMC BANK 0 (ADC)/ADCIO_16
- net Net-(J9-PadG06) renamed /FMC BANK 0 (ADC)/RFMC_I2C_SCL
- net Net-(J9-PadG21) renamed /FMC BANK 0 (ADC)/VCM01_227
- net Net-(J9-PadG35) renamed /FMC BANK 0 (ADC)/ADC_CLKIN_1_P
- net Net-(J9-PadG38) renamed /FMC BANK 0 (ADC)/ADC_CLKIN_3_P
- net Net-(J9-PadH01) renamed /FMC BANK 0 (ADC)/ADCIO_17
- net Net-(J9-PadH03) renamed /FMC BANK 0 (ADC)/ADCIO_18
- net Net-(J9-PadH05) renamed /FMC BANK 0 (ADC)/ADCIO_19
- net Net-(J9-PadH21) renamed /FMC BANK 0 (ADC)/VCM23_227
- J10 pad A01: Net-(J10-PadA01) -> /FMC BANK 1 (DAC)/VCC12_SW
- J10 pad A34: Net-(J10-PadA34) -> /FMC BANK 1 (DAC)/UTIL_3V3
- J10 pad A35: Net-(J10-PadA35) -> /FMC BANK 1 (DAC)/VCC1V8_BUS
- J10 pad A36: Net-(J10-PadA36) -> GND
- J10 pad A38: Net-(J10-PadA38) -> GND
- J10 pad A40: Net-(J10-PadA40) -> GND
- J10 pad B01: Net-(J10-PadB01) -> /FMC BANK 1 (DAC)/VCC12_SW
- J10 pad B02: Net-(J10-PadB02) -> GND
- J10 pad B03: Net-(J10-PadB03) -> GND
- J10 pad B05: Net-(J10-PadB05) -> GND
- J10 pad B06: Net-(J10-PadB06) -> GND
- J10 pad B08: Net-(J10-PadB08) -> GND
- J10 pad B09: Net-(J10-PadB09) -> GND
- J10 pad B11: Net-(J10-PadB11) -> GND
- J10 pad B12: Net-(J10-PadB12) -> GND
- J10 pad B22: DAC_D0_P -> unconnected-(J10-PadB22)
- J10 pad B25: DAC_C0_P -> unconnected-(J10-PadB25)
- J10 pad B28: Net-(J10-PadB28) -> unconnected-(J10-PadB28)
- J10 pad B29: Net-(J10-PadB29) -> GND
- J10 pad B30: Net-(J10-PadB30) -> GND
- J10 pad B31: Net-(J10-PadB31) -> unconnected-(J10-PadB31)
- J10 pad B32: Net-(J10-PadB32) -> GND
- J10 pad B33: Net-(J10-PadB33) -> GND
- J10 pad B34: Net-(J10-PadB34) -> /FMC BANK 1 (DAC)/UTIL_3V3
- J10 pad B35: Net-(J10-PadB35) -> GND
- J10 pad B37: Net-(J10-PadB37) -> GND
- J10 pad B39: Net-(J10-PadB39) -> GND
- J10 pad C01: Net-(J10-PadC01) -> /FMC BANK 1 (DAC)/VCC12_SW
- J10 pad C02: Net-(J10-PadC02) -> GND
- J10 pad C03: Net-(J10-PadC03) -> GND
- J10 pad C05: Net-(J10-PadC05) -> GND
- J10 pad C06: Net-(J10-PadC06) -> GND
- J10 pad C08: Net-(J10-PadC08) -> GND
- J10 pad C09: Net-(J10-PadC09) -> GND
- J10 pad C11: Net-(J10-PadC11) -> GND
- J10 pad C12: Net-(J10-PadC12) -> GND
- J10 pad C22: DAC_D0_N -> unconnected-(J10-PadC22)
- J10 pad C25: DAC_C0_N -> unconnected-(J10-PadC25)
- J10 pad C28: Net-(J10-PadC28) -> unconnected-(J10-PadC28)
- J10 pad C29: Net-(J10-PadC29) -> GND
- J10 pad C30: Net-(J10-PadC30) -> GND
- J10 pad C31: Net-(J10-PadC31) -> unconnected-(J10-PadC31)
- J10 pad C32: Net-(J10-PadC32) -> GND
- J10 pad C33: Net-(J10-PadC33) -> GND
- J10 pad C34: Net-(J10-PadC34) -> /FMC BANK 1 (DAC)/UTIL_3V3
- J10 pad C35: Net-(J10-PadC35) -> /FMC BANK 1 (DAC)/VCC1V8_BUS
- J10 pad C36: Net-(J10-PadC36) -> GND
- J10 pad C38: Net-(J10-PadC38) -> GND
- J10 pad C40: Net-(J10-PadC40) -> GND
- J10 pad D01: Net-(J10-PadD01) -> /FMC BANK 1 (DAC)/VCC12_SW
- J10 pad D34: Net-(J10-PadD34) -> /FMC BANK 1 (DAC)/UTIL_3V3
- J10 pad D35: Net-(J10-PadD35) -> GND
- J10 pad D37: Net-(J10-PadD37) -> GND
- J10 pad D39: Net-(J10-PadD39) -> GND
- J10 pad E01: Net-(J10-PadE01) -> /FMC BANK 1 (DAC)/VCC12_SW
- J10 pad E34: Net-(J10-PadE34) -> /FMC BANK 1 (DAC)/UTIL_3V3
- J10 pad E35: Net-(J10-PadE35) -> unconnected-(J10-PadE35)
- J10 pad E36: Net-(J10-PadE36) -> GND
- J10 pad E38: Net-(J10-PadE38) -> GND
- J10 pad E40: Net-(J10-PadE40) -> GND
- J10 pad F01: Net-(J10-PadF01) -> GND
- J10 pad F02: Net-(J10-PadF02) -> GND
- J10 pad F03: Net-(J10-PadF03) -> GND
- J10 pad F04: Net-(J10-PadF04) -> GND
- J10 pad F06: Net-(J10-PadF06) -> GND
- J10 pad F07: Net-(J10-PadF07) -> GND
- J10 pad F09: Net-(J10-PadF09) -> GND
- J10 pad F10: Net-(J10-PadF10) -> GND
- J10 pad F12: Net-(J10-PadF12) -> GND
- J10 pad F13: Net-(J10-PadF13) -> GND
- J10 pad F23: DAC_D1_P -> unconnected-(J10-PadF23)
- J10 pad F26: DAC_C1_P -> unconnected-(J10-PadF26)
- J10 pad F29: Net-(J10-PadF29) -> unconnected-(J10-PadF29)
- J10 pad F30: Net-(J10-PadF30) -> GND
- J10 pad F31: Net-(J10-PadF31) -> GND
- J10 pad F32: Net-(J10-PadF32) -> unconnected-(J10-PadF32)
- J10 pad F33: Net-(J10-PadF33) -> GND
- J10 pad F34: Net-(J10-PadF34) -> GND
- J10 pad F35: Net-(J10-PadF35) -> GND
- J10 pad F37: Net-(J10-PadF37) -> GND
- J10 pad F39: Net-(J10-PadF39) -> GND
- J10 pad G01: Net-(J10-PadG01) -> /FMC BANK 1 (DAC)/DAC_AVTT_BUS
- J10 pad G02: Net-(J10-PadG02) -> /FMC BANK 1 (DAC)/DAC_AVTT_BUS
- J10 pad G03: Net-(J10-PadG03) -> GND
- J10 pad G04: Net-(J10-PadG04) -> GND
- J10 pad G06: Net-(J10-PadG06) -> GND
- J10 pad G07: Net-(J10-PadG07) -> GND
- J10 pad G09: Net-(J10-PadG09) -> GND
- J10 pad G10: Net-(J10-PadG10) -> GND
- J10 pad G12: Net-(J10-PadG12) -> GND
- J10 pad G13: Net-(J10-PadG13) -> GND
- J10 pad G23: DAC_D1_N -> unconnected-(J10-PadG23)
- J10 pad G26: DAC_C1_N -> unconnected-(J10-PadG26)
- J10 pad G29: Net-(J10-PadG29) -> unconnected-(J10-PadG29)
- J10 pad G30: Net-(J10-PadG30) -> GND
- J10 pad G31: Net-(J10-PadG31) -> GND
- J10 pad G32: Net-(J10-PadG32) -> unconnected-(J10-PadG32)
- J10 pad G33: Net-(J10-PadG33) -> GND
- J10 pad G34: Net-(J10-PadG34) -> GND
- J10 pad G35: Net-(J10-PadG35) -> unconnected-(J10-PadG35)
- J10 pad G36: Net-(J10-PadG36) -> GND
- J10 pad G38: Net-(J10-PadG38) -> GND
- J10 pad G40: Net-(J10-PadG40) -> GND
- J10 pad H01: Net-(J10-PadH01) -> /FMC BANK 1 (DAC)/DAC_AVTT_BUS
- J10 pad H02: GND -> /FMC BANK 1 (DAC)/DAC_AVTT_BUS
- J10 pad H34: Net-(J10-PadH34) -> /FMC BANK 1 (DAC)/UTIL_3V3
- J10 pad H35: Net-(J10-PadH35) -> GND
- J10 pad H37: Net-(J10-PadH37) -> GND
- J10 pad H39: Net-(J10-PadH39) -> GND
- J9 pad A01: Net-(J9-PadA01) -> GND
- J9 pad A03: Net-(J9-PadA03) -> GND
- J9 pad A05: Net-(J9-PadA05) -> GND
- J9 pad A06: Net-(J9-PadA06) -> /FMC BANK 0 (ADC)/VCC1V8_BUS
- J9 pad A07: Net-(J9-PadA07) -> /FMC BANK 0 (ADC)/UTIL_3V3
- J9 pad B02: Net-(J9-PadB02) -> GND
- J9 pad B04: Net-(J9-PadB04) -> GND
- J9 pad B05: Net-(J9-PadB05) -> /FMC BANK 0 (ADC)/ADCIO_05
- J9 pad B06: Net-(J9-PadB06) -> GND
- J9 pad B07: Net-(J9-PadB07) -> GND
- J9 pad B21: GND -> /FMC BANK 0 (ADC)/VCM23_224
- J9 pad B22: Net-(J9-PadB22) -> GND
- J9 pad B23: Net-(J9-PadB23) -> GND
- J9 pad B24: Net-(J9-PadB24) -> unconnected-(J9-PadB24)
- J9 pad B25: Net-(J9-PadB25) -> GND
- J9 pad B26: Net-(J9-PadB26) -> GND
- J9 pad B27: Net-(J9-PadB27) -> unconnected-(J9-PadB27)
- J9 pad B28: Net-(J9-PadB28) -> GND
- J9 pad B29: Net-(J9-PadB29) -> GND
- J9 pad B30: Net-(J9-PadB30) -> unconnected-(J9-PadB30)
- J9 pad B31: Net-(J9-PadB31) -> GND
- J9 pad B32: Net-(J9-PadB32) -> GND
- J9 pad B33: Net-(J9-PadB33) -> unconnected-(J9-PadB33)
- J9 pad B34: Net-(J9-PadB34) -> GND
- J9 pad B35: Net-(J9-PadB35) -> GND
- J9 pad B37: Net-(J9-PadB37) -> GND
- J9 pad B38: Net-(J9-PadB38) -> GND
- J9 pad B40: Net-(J9-PadB40) -> GND
- J9 pad C01: Net-(J9-PadC01) -> GND
- J9 pad C02: Net-(J9-PadC02) -> /FMC BANK 0 (ADC)/ADCIO_05
- J9 pad C03: Net-(J9-PadC03) -> GND
- J9 pad C05: Net-(J9-PadC05) -> GND
- J9 pad C06: Net-(J9-PadC06) -> /FMC BANK 0 (ADC)/VCC1V8_BUS
- J9 pad C07: Net-(J9-PadC07) -> /FMC BANK 0 (ADC)/UTIL_3V3
- J9 pad C21: GND -> /FMC BANK 0 (ADC)/VCM01_225
- J9 pad C22: Net-(J9-PadC22) -> GND
- J9 pad C23: Net-(J9-PadC23) -> GND
- J9 pad C24: Net-(J9-PadC24) -> unconnected-(J9-PadC24)
- J9 pad C25: Net-(J9-PadC25) -> GND
- J9 pad C26: Net-(J9-PadC26) -> GND
- J9 pad C27: Net-(J9-PadC27) -> unconnected-(J9-PadC27)
- J9 pad C28: Net-(J9-PadC28) -> GND
- J9 pad C29: Net-(J9-PadC29) -> GND
- J9 pad C30: Net-(J9-PadC30) -> unconnected-(J9-PadC30)
- J9 pad C31: Net-(J9-PadC31) -> GND
- J9 pad C32: Net-(J9-PadC32) -> GND
- J9 pad C33: Net-(J9-PadC33) -> unconnected-(J9-PadC33)
- J9 pad C34: Net-(J9-PadC34) -> GND
- J9 pad C35: Net-(J9-PadC35) -> GND
- J9 pad C37: Net-(J9-PadC37) -> GND
- J9 pad C38: Net-(J9-PadC38) -> GND
- J9 pad C40: Net-(J9-PadC40) -> GND
- J9 pad D02: Net-(J9-PadD02) -> GND
- J9 pad D04: Net-(J9-PadD04) -> GND
- J9 pad D06: Net-(J9-PadD06) -> GND
- J9 pad D07: Net-(J9-PadD07) -> /FMC BANK 0 (ADC)/UTIL_3V3
- J9 pad E01: Net-(J9-PadE01) -> GND
- J9 pad E03: Net-(J9-PadE03) -> GND
- J9 pad E05: Net-(J9-PadE05) -> GND
- J9 pad E07: Net-(J9-PadE07) -> /FMC BANK 0 (ADC)/UTIL_3V3
- J9 pad F02: Net-(J9-PadF02) -> GND
- J9 pad F04: Net-(J9-PadF04) -> GND
- J9 pad F06: Net-(J9-PadF06) -> GND
- J9 pad F07: Net-(J9-PadF07) -> /FMC BANK 0 (ADC)/UTIL_3V3
- J9 pad F22: Net-(J9-PadF22) -> GND
- J9 pad F23: Net-(J9-PadF23) -> unconnected-(J9-PadF23)
- J9 pad F24: Net-(J9-PadF24) -> GND
- J9 pad F25: Net-(J9-PadF25) -> GND
- J9 pad F26: Net-(J9-PadF26) -> unconnected-(J9-PadF26)
- J9 pad F27: Net-(J9-PadF27) -> GND
- J9 pad F28: Net-(J9-PadF28) -> GND
- J9 pad F29: Net-(J9-PadF29) -> unconnected-(J9-PadF29)
- J9 pad F30: Net-(J9-PadF30) -> GND
- J9 pad F31: Net-(J9-PadF31) -> GND
- J9 pad F32: Net-(J9-PadF32) -> unconnected-(J9-PadF32)
- J9 pad F33: Net-(J9-PadF33) -> GND
- J9 pad F34: Net-(J9-PadF34) -> GND
- J9 pad F36: Net-(J9-PadF36) -> GND
- J9 pad F37: Net-(J9-PadF37) -> GND
- J9 pad F39: Net-(J9-PadF39) -> GND
- J9 pad F40: Net-(J9-PadF40) -> GND
- J9 pad G01: Net-(J9-PadG01) -> GND
- J9 pad G03: Net-(J9-PadG03) -> GND
- J9 pad G05: Net-(J9-PadG05) -> GND
- J9 pad G07: Net-(J9-PadG07) -> /FMC BANK 0 (ADC)/UTIL_3V3
- J9 pad G22: Net-(J9-PadG22) -> GND
- J9 pad G23: Net-(J9-PadG23) -> unconnected-(J9-PadG23)
- J9 pad G24: Net-(J9-PadG24) -> GND
- J9 pad G25: Net-(J9-PadG25) -> GND
- J9 pad G26: Net-(J9-PadG26) -> unconnected-(J9-PadG26)
- J9 pad G27: Net-(J9-PadG27) -> GND
- J9 pad G28: Net-(J9-PadG28) -> GND
- J9 pad G29: Net-(J9-PadG29) -> unconnected-(J9-PadG29)
- J9 pad G30: Net-(J9-PadG30) -> GND
- J9 pad G31: Net-(J9-PadG31) -> GND
- J9 pad G32: Net-(J9-PadG32) -> unconnected-(J9-PadG32)
- J9 pad G33: Net-(J9-PadG33) -> GND
- J9 pad G34: Net-(J9-PadG34) -> GND
- J9 pad G36: Net-(J9-PadG36) -> GND
- J9 pad G37: Net-(J9-PadG37) -> GND
- J9 pad G39: Net-(J9-PadG39) -> GND
- J9 pad G40: Net-(J9-PadG40) -> GND
- J9 pad H02: Net-(J9-PadH02) -> GND
- J9 pad H04: Net-(J9-PadH04) -> GND
- J9 pad H06: Net-(J9-PadH06) -> GND
- J9 pad H07: Net-(J9-PadH07) -> /FMC BANK 0 (ADC)/UTIL_3V3
- U1 pad 1: Net-(U1-Pad1) -> unconnected-(U1-Pad1)
- U2 pad 1: Net-(U2-Pad1) -> unconnected-(U2-Pad1)
- U3 pad 1: Net-(U3-Pad1) -> unconnected-(U3-Pad1)
- U4 pad 1: Net-(U4-Pad1) -> unconnected-(U4-Pad1)
- U5 pad 1: Net-(U5-Pad1) -> unconnected-(U5-Pad1)
- U6 pad 1: Net-(U6-Pad1) -> unconnected-(U6-Pad1)
- U7 pad 1: Net-(U7-Pad1) -> unconnected-(U7-Pad1)
- U8 pad 1: Net-(U8-Pad1) -> unconnected-(U8-Pad1)
Routing:
- net Net-(J2-Pad1): track 6.67 -> 7.36 mm
- net DAC_B1_P: track 31.6 -> 30.9 mm, vias 2 -> 1
- net Net-(J1-Pad1): track 6.73 -> 7.36 mm
- net DAC_B0_P: track 13.6 -> 13.3 mm, vias 2 -> 1
- net ADC_A0_P: vias 2 -> 1
- net ADC_A0_N: vias 2 -> 1
- net DAC_A1_P: vias 2 -> 1
- net ADC_A1_P: vias 2 -> 1
- net DAC_B1_N: vias 2 -> 1
- net DAC_B0_N: vias 2 -> 1
- net DAC_A1_N: vias 2 -> 1
- net DAC_A0_N: vias 2 -> 1
- net ADC_B1_P: vias 2 -> 1
- net ADC_B0_N: vias 2 -> 1
- net ADC_B0_P: vias 2 -> 1
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Other:
- outline, holes or cut-outs redrawn
- board text added: "1"
- board text added: "10"
- board text added: "15"
- board text added: "20"
- board text added: "25"
- board text added: "30"
- board text added: "35"
- board text added: "40"
- board text added: "5"
- board text added: "A"
- board text added: "ADC224 PAIR 0,1 (CHANNEL 0 I/Q)"
- board text added: "ADC225 PAIR 0,1 (CHANNEL 1 I/Q)"
- board text added: "B"
- board text added: "B10"
- board text added: "B13"
- board text added: "B16"
- board text added: "B19"
- board text added: "B19,C19 RFMC_DAC_06"
- board text added: "C"
- board text added: "C10"
- board text added: "C13"
- board text added: "C16"
- board text added: "C19"
- board text added: "D"
- board text added: "DAC229 PAIR 0,1 (CHANNEL 1 I/Q)"
- board text added: "DAC229 PAIR 2,3 (CHANNEL 0 I/Q)"
- board text added: "E"
- board text added: "F"
- board text added: "F09"
- board text added: "F12"
- board text added: "F17"
- board text added: "F20"
- board text added: "F20,G20 RFMC_ADC_07"
- board text added: "FORK 'EM"
- board text added: "G"
- board text added: "G09"
- board text added: "G12"
- board text added: "G17"
- board text added: "G20"
- board text added: "H"
- board text added: "RFMC ADC"
- board text added: "RFMC DAC"
- board text added: "Ryan Stephenson Cody Roberson Eric Weeks Arizona State University"
